File: Rocket Sensor Board/Sensor Board.brd (EAGLE design)
At the start: 38.5 x 66 mm, 115 parts, among them J1 501568-0207, J2 501568-0207, J3 SD-105027-101, J4 501568-0407, U1 MAG3110, U10 ADXL362, U11 TM4C1233H6PM, U12 TPS62082DSGR, U13 SN74AUP3G17, U15 ADT7301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

Commit message: Rocket Sensor Board: Changed passives on LIS3DH, H3LIS331DLTR, L3GD20H, LSM303D, LSM9DS0, ADXL362 (But not the Tantalum), MAX2100 and Si7013 to use the new library parts with full documentaion and part numbers
Parts:
- removed C54: 10uF, Kas-Passives:4.3X7.3SMD
- added C57: 0.1 uF, Kas-Passives:C0402
- added C58, C59, C60: 10uF, Kas-Passives:C0603
- C10: value 10nF -> 0.01 uF
- C11: value 1uF -> 0.1 uF
- C12: value 10uF -> 0.1 uF
- C13: value 100nF -> 10uF; device Kas-Passives:4.3X7.3SMD -> Kas-Passives:C0603
- C14, C20, C26, C27, C8, C9: value 100nF -> 0.1 uF
- C18, C21, C48: device Kas-Passives:C0402 -> Kas-Passives:C0603
- C22, C45, C47: value 10uF -> 0.1 uF; device Kas-Passives:4.3X7.3SMD -> Kas-Passives:C0402
- C25, C46, C7: device Kas-Passives:4.3X7.3SMD -> Kas-Passives:C0603
- C28, C29, C6: value 0.1uF -> 0.1 uF
- C51: value (none) -> 4.7 uF
- moved C22 117.9 mm to (-14.1, -52.5), flipped to the top, turned to 0 degrees
- moved C46 110.1 mm to (-14.2, -48.9), flipped to the top, turned to 0 degrees
- moved C25 109.2 mm to (-14.2, -44.1), flipped to the top, turned to 0 degrees
- moved C7 76.6 mm to (-14.2, -19.3), flipped to the top
- moved C47 70.7 mm to (-14.1, -23.0), flipped to the top, turned to 0 degrees
- moved C13 70.5 mm to (-14.2, -31.7), flipped to the top, turned to 0 degrees
- moved C45 65.3 mm to (-14.1, -35.4), flipped to the top, turned to 0 degrees
Connections:
- net 3.3V-A: now also C13.2, C22.2, C25.1, C45.2, C46.1, C47.2, C57.1, C58.2, C59.2, C60.2, C7.1; no longer C13.P$1, C22.P$2, C25.P$1, C45.P$1, C46.P$1, C47.P$1, C54.P$1, C7.P$1
- net GND: now also C13.1, C22.1, C25.2, C45.1, C46.2, C47.1, C57.2, C58.1, C59.1, C60.1, C7.2; no longer C13.P$2, C22.P$1, C25.P$2, C45.P$2, C46.P$2, C47.P$2, C54.P$2, C7.P$2
Routing:
- net GND: track 59.2 -> 45.8 mm
- net 3.3V-A: track 239.0 -> 227.7 mm
