File: FRDM-KL25 SD Card - Battery Board/SD Card - Battery Board.sch (EAGLE design)
At the start: 59 parts, among them U1 TPS63001, U2 TPS63002, U3 BQ27510DRZT-G3, U4 BQ24210DQCT

Commit message: FRDM-KL25Z: Corrected part names
Parts:
- removed U$1: (no value), Kas-Diodes-LEDs:SCHOTTKY
- added D1: Yellow-LED, Kas-Diodes-LEDs:1.6X3.2Y-X.XX-XXMA
- D3: value Yellow-LED -> (none); device Kas-Diodes-LEDs:1.6X3.2Y-X.XX-XXMA -> Kas-Diodes-LEDs:SCHOTTKY
- renumbered U$2 to D4, U$3 to J2
Other:
- moved on the sheet: D3
Changed lines of the file:
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@@
 <part name="R25" library="Kas-Resistors" deviceset="RESISTOR" device="10K-63M-1%-50V" value="10k"/>
 <part name="R26" library="Kas-Resistors" deviceset="RESISTOR" device="1K-62.5M-0.1%-75V" value="1k"/>
-<part name="D3" library="Kas-Diodes-LEDs" deviceset="1.6X3.2" device="Y-X.XX-XXMA" value="Yellow-LED"/>
+<part name="D1" library="Kas-Diodes-LEDs" deviceset="1.6X3.2" device="Y-X.XX-XXMA" value="Yellow-LED"/>
 <part name="J1" library="Kas-Connectors" deviceset="SD_CARD_SLOT" device=""/>
 <part name="C2" library="Kas-Capacitors" deviceset="CAPACITOR" device="10U-X7R-10%-6.3V" value="10uF"/>
@@
 <part name="C11" library="Kas-Capacitors" deviceset="CAPACITOR" device="0.1U-X5R-10%25V-0603" value="0.1uF"/>
 <part name="C12" library="Kas-Capacitors" deviceset="CAPACITOR" device="0.1U-X5R-10%25V-0603" value="0.1uF"/>
-<part name="U$1" library="Kas-Diodes-LEDs" deviceset="SCHOTTKY" device=""/>
-<part name="U$2" library="Kas-Diodes-LEDs" deviceset="SCHOTTKY" device=""/>
-<part name="U$3" library="Kas-Connectors" deviceset="USB-MICRO" device="SD-47346-001"/>
+<part name="D3" library="Kas-Diodes-LEDs" deviceset="SCHOTTKY" device=""/>
+<part name="D4" library="Kas-Diodes-LEDs" deviceset="SCHOTTKY" device=""/>
+<part name="J2" library="Kas-Connectors" deviceset="USB-MICRO" device="SD-47346-001"/>
 <part name="R27" library="Kas-Resistors" deviceset="RESISTOR" device="0-100M-X%-50V" value="0"/>
 <part name="R28" library="Kas-Resistors" deviceset="RESISTOR" device="0-100M-X%-50V" value="0"/>
@@
 <instance part="R25" gate="G$1" x="124.46" y="-20.32"/>
 <instance part="R26" gate="G$1" x="132.08" y="-5.08"/>
-<instance part="D3" gate="G$1" x="127" y="10.16" rot="R180"/>
+<instance part="D1" gate="G$1" x="127" y="10.16" rot="R180"/>
 <instance part="C2" gate="G$1" x="-43.18" y="106.68"/>
 <instance part="C3" gate="G$1" x="-43.18" y="71.12"/>
@@
 <instance part="C11" gate="G$1" x="165.1" y="45.72"/>
 <instance part="C12" gate="G$1" x="180.34" y="33.02"/>
-<instance part="U$1" gate="G$1" x="25.4" y="91.44"/>
-<instance part="U$2" gate="G$1" x="17.78" y="17.78"/>
-<instance part="U$3" gate="G$1" x="2.54" y="-43.18"/>
+<instance part="D3" gate="G$1" x="25.4" y="91.44"/>
+<instance part="D4" gate="G$1" x="17.78" y="17.78"/>
+<instance part="J2" gate="G$1" x="2.54" y="-43.18"/>
 <instance part="R27" gate="G$1" x="22.86" y="73.66"/>
 <instance part="R28" gate="G$1" x="17.78" y="0"/>

Commit message: FRDM-KL25Z: Corrected all parts to be found and avilable at newark, packages where corrected as needed BOM should now be correct, one final check needed before ordering parts
Parts:
- C1, C9: device Kas-Capacitors:CAPACITOR0.47U-X5R-10%-6.3V-0603 -> Kas-Capacitors:CAPACITOR0.47U-X5R-10%-10V-0603
- C13, C14: device Kas-Capacitors:CAPACITOR0.1U-X7R-10%-10V -> Kas-Capacitors:CAPACITOR0.1U-X7R-10%-25V-0603
- R1, R11, R12, R13, R18, R19, R2, R20, R21, R24, R25, R3, R4, R5, R6, R7, R8: device Kas-Resistors:RESISTOR10K-63M-1%-50V -> Kas-Resistors:RESISTOR10K-100M-0.5%-75V
- R17: device Kas-Resistors:RESISTOR0-100M-X%-50V -> Kas-Resistors:RESISTOR0.01-100M-1%-50V
Changed lines of the file:
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@@
 </classes>
 <parts>
-<part name="R1" library="Kas-Resistors" deviceset="RESISTOR" device="10K-63M-1%-50V" value="10k"/>
-<part name="R2" library="Kas-Resistors" deviceset="RESISTOR" device="10K-63M-1%-50V" value="10k"/>
-<part name="R3" library="Kas-Resistors" deviceset="RESISTOR" device="10K-63M-1%-50V" value="10k"/>
-<part name="R4" library="Kas-Resistors" deviceset="RESISTOR" device="10K-63M-1%-50V" value="10k"/>
-<part name="R5" library="Kas-Resistors" deviceset="RESISTOR" device="10K-63M-1%-50V" value="10k"/>
-<part name="R6" library="Kas-Resistors" deviceset="RESISTOR" device="10K-63M-1%-50V" value="10k"/>
-<part name="R7" library="Kas-Resistors" deviceset="RESISTOR" device="10K-63M-1%-50V" value="10k"/>
-<part name="R8" library="Kas-Resistors" deviceset="RESISTOR" device="10K-63M-1%-50V" value="10k"/>
+<part name="R1" library="Kas-Resistors" deviceset="RESISTOR" device="10K-100M-0.5%-75V" value="10k"/>
+<part name="R2" library="Kas-Resistors" deviceset="RESISTOR" device="10K-100M-0.5%-75V" value="10k"/>
+<part name="R3" library="Kas-Resistors" deviceset="RESISTOR" device="10K-100M-0.5%-75V" value="10k"/>
+<part name="R4" library="Kas-Resistors" deviceset="RESISTOR" device="10K-100M-0.5%-75V" value="10k"/>
+<part name="R5" library="Kas-Resistors" deviceset="RESISTOR" device="10K-100M-0.5%-75V" value="10k"/>
+<part name="R6" library="Kas-Resistors" deviceset="RESISTOR" device="10K-100M-0.5%-75V" value="10k"/>
+<part name="R7" library="Kas-Resistors" deviceset="RESISTOR" device="10K-100M-0.5%-75V" value="10k"/>
+<part name="R8" library="Kas-Resistors" deviceset="RESISTOR" device="10K-100M-0.5%-75V" value="10k"/>
 <part name="R9" library="Kas-Resistors" deviceset="RESISTOR" device="200-100M-0.1%-75V" value="200"/>
 <part name="R10" library="Kas-Resistors" deviceset="RESISTOR" device="200-100M-0.1%-75V" value="200"/>
@@
 <part name="U4" library="Kas-Buck Boost Battery Control" deviceset="B224210" device="" value="BQ24210DQCT"/>
 <part name="GND1" library="supply1" deviceset="GND" device=""/>
-<part name="R11" library="Kas-Resistors" deviceset="RESISTOR" device="10K-63M-1%-50V" value="10k"/>
-<part name="R12" library="Kas-Resistors" deviceset="RESISTOR" device="10K-63M-1%-50V" value="10k"/>
-<part name="R13" library="Kas-Resistors" deviceset="RESISTOR" device="10K-63M-1%-50V" value="10k"/>
+<part name="R11" library="Kas-Resistors" deviceset="RESISTOR" device="10K-100M-0.5%-75V" value="10k"/>
+<part name="R12" library="Kas-Resistors" deviceset="RESISTOR" device="10K-100M-0.5%-75V" value="10k"/>
+<part name="R13" library="Kas-Resistors" deviceset="RESISTOR" device="10K-100M-0.5%-75V" value="10k"/>
 <part name="D2" library="Kas-Diodes-LEDs" deviceset="1.6X3.2" device="R-1.85V-20MA" value="Red-LED"/>
 <part name="R14" library="Kas-Resistors" deviceset="RESISTOR" device="1K-62.5M-0.1%-75V" value="1k"/>
@@
 <part name="GND3" library="supply1" deviceset="GND" device=""/>
 <part name="R16" library="Kas-Resistors" deviceset="RESISTOR" device="100-62.5M-0.1%-75V" value="100"/>
-<part name="R17" library="Kas-Resistors" deviceset="RESISTOR" device="0-100M-X%-50V" value="0.01"/>
-<part name="R18" library="Kas-Resistors" deviceset="RESISTOR" device="10K-63M-1%-50V" value="10k"/>
-<part name="R19" library="Kas-Resistors" deviceset="RESISTOR" device="10K-63M-1%-50V" value="10k"/>
-<part name="R20" library="Kas-Resistors" deviceset="RESISTOR" device="10K-63M-1%-50V" value="10k"/>
-<part name="R21" library="Kas-Resistors" deviceset="RESISTOR" device="10K-63M-1%-50V" value="10k"/>
+<part name="R17" library="Kas-Resistors" deviceset="RESISTOR" device="0.01-100M-1%-50V" value="0.01"/>
+<part name="R18" library="Kas-Resistors" deviceset="RESISTOR" device="10K-100M-0.5%-75V" value="10k"/>
+<part name="R19" library="Kas-Resistors" deviceset="RESISTOR" device="10K-100M-0.5%-75V" value="10k"/>
+<part name="R20" library="Kas-Resistors" deviceset="RESISTOR" device="10K-100M-0.5%-75V" value="10k"/>
+<part name="R21" library="Kas-Resistors" deviceset="RESISTOR" device="10K-100M-0.5%-75V" value="10k"/>
 <part name="R22" library="Kas-Resistors" deviceset="RESISTOR" device="1.6K-125M-0.1%-100V" value="1.6k"/>
 <part name="R23" library="Kas-Resistors" deviceset="RESISTOR" device="20K-63M-1%-50V" value="20k"/>
-<part name="R24" library="Kas-Resistors" deviceset="RESISTOR" device="10K-63M-1%-50V" value="10k"/>
-<part name="R25" library="Kas-Resistors" deviceset="RESISTOR" device="10K-63M-1%-50V" value="10k"/>
+<part name="R24" library="Kas-Resistors" deviceset="RESISTOR" device="10K-100M-0.5%-75V" value="10k"/>
+<part name="R25" library="Kas-Resistors" deviceset="RESISTOR" device="10K-100M-0.5%-75V" value="10k"/>
 <part name="R26" library="Kas-Resistors" deviceset="RESISTOR" device="1K-62.5M-0.1%-75V" value="1k"/>
 <part name="D1" library="Kas-Diodes-LEDs" deviceset="1.6X3.2" device="Y-X.XX-XXMA" value="Yellow-LED"/>
@@
 <part name="C7" library="Kas-Capacitors" deviceset="CAPACITOR" device="0.1U-X7R-10%-25V" value="0.1uF"/>
 <part name="C8" library="Kas-Capacitors" deviceset="CAPACITOR" device="1U-X5R-10%-10V-0603" value="1uF"/>
-<part name="C1" library="Kas-Capacitors" deviceset="CAPACITOR" device="0.47U-X5R-10%-6.3V-0603" value="0.47uF"/>
-<part name="C9" library="Kas-Capacitors" deviceset="CAPACITOR" device="0.47U-X5R-10%-6.3V-0603" value="0.47uF"/>
+<part name="C1" library="Kas-Capacitors" deviceset="CAPACITOR" device="0.47U-X5R-10%-10V-0603" value="0.47uF"/>
+<part name="C9" library="Kas-Capacitors" deviceset="CAPACITOR" device="0.47U-X5R-10%-10V-0603" value="0.47uF"/>
 <part name="C10" library="Kas-Capacitors" deviceset="CAPACITOR" device="0.1U-X5R-10%25V-0603" value="0.1uF"/>
 <part name="C11" library="Kas-Capacitors" deviceset="CAPACITOR" device="0.1U-X5R-10%25V-0603" value="0.1uF"/>
@@
 <part name="R32" library="Kas-Resistors" deviceset="RESISTOR" device="100-62.5M-0.1%-75V" value="100"/>
 <part name="R33" library="Kas-Resistors" deviceset="RESISTOR" device="100-62.5M-0.1%-75V" value="100"/>
-<part name="C13" library="Kas-Capacitors" deviceset="CAPACITOR" device="0.1U-X7R-10%-10V" value="0.1uF"/>
-<part name="C14" library="Kas-Capacitors" deviceset="CAPACITOR" device="0.1U-X7R-10%-10V" value="0.1uF"/>
+<part name="C13" library="Kas-Capacitors" deviceset="CAPACITOR" device="0.1U-X7R-10%-25V-0603" value="0.1uF"/>
+<part name="C14" library="Kas-Capacitors" deviceset="CAPACITOR" device="0.1U-X7R-10%-25V-0603" value="0.1uF"/>
 </parts>
 <sheets>
